File: PCB Files/Reflowduino Pro/Reflowduino Pro v2.brd (EAGLE design)
At the start: 86.4 x 53.3 mm, 57 parts, among them IC1 MCP73831, IC2 ATMEGA32U4, IC3 AP2112K-3.3TRG1, IC4 MAX31855, J1 microUSB, J10 RLY-, J2 LiPo Battery, J5 Thermocouple, J6 ICSP, J9 RLY+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

Commit message: Add files via upload
Other:
- board text added: "Designed by Timothy Woo Hardware released under CC-BY-SA-4.0 license"
- board text removed: "Designed by Timothy Woo"
Changed lines of the file:
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@@
 <layer number="23" name="tOrigins" color="15" fill="1" visible="yes" active="yes"/>
 <layer number="24" name="bOrigins" color="15" fill="1" visible="yes" active="yes"/>
-<layer number="25" name="tNames" color="7" fill="1" visible="no" active="yes"/>
+<layer number="25" name="tNames" color="7" fill="1" visible="yes" active="yes"/>
 <layer number="26" name="bNames" color="7" fill="1" visible="no" active="yes"/>
 <layer number="27" name="tValues" color="7" fill="1" visible="no" active="yes"/>
@@
 <wire x1="58.42" y1="5.08" x2="55.88" y2="2.54" width="0.3048" layer="21"/>
 <wire x1="55.88" y1="2.54" x2="55.88" y2="0" width="0.3048" layer="21"/>
-<text x="1.27" y="57.15" size="2.1844" layer="25" font="vector" ratio="16">Designed by Timothy Woo</text>
+<text x="1.27" y="57.15" size="2.1844" layer="51" font="vector" ratio="16">Designed by Timothy Woo
+Hardware released under CC-BY-SA-4.0 license</text>
 <text x="14.5415" y="31.3055" size="0.8128" layer="21" font="vector" ratio="16">DONE</text>
 <text x="9.525" y="10.16" size="1.27" layer="21" font="vector" ratio="16">+</text>

Commit message: Add files via upload
Other:
- board text added: "Designed by Timothy Woo Released under CC-BY-SA-4.0 license"
- board text removed: "Designed by Timothy Woo Hardware released under CC-BY-SA-4.0 license"
Changed lines of the file:
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@@
 <wire x1="55.88" y1="2.54" x2="55.88" y2="0" width="0.3048" layer="21"/>
 <text x="1.27" y="57.15" size="2.1844" layer="51" font="vector" ratio="16">Designed by Timothy Woo
-Hardware released under CC-BY-SA-4.0 license</text>
+Released under CC-BY-SA-4.0 license</text>
 <text x="14.5415" y="31.3055" size="0.8128" layer="21" font="vector" ratio="16">DONE</text>
 <text x="9.525" y="10.16" size="1.27" layer="21" font="vector" ratio="16">+</text>
