File: PCB Files/Reflowduino Pro/Reflowduino Pro v2.brd (EAGLE design)
At the start: 86.4 x 53.3 mm, 57 parts, among them IC1 MCP73831, IC2 ATMEGA32U4, IC3 AP2112K-3.3TRG1, IC4 MAX31855, J1 microUSB, J10 RLY-, J2 LiPo Battery, J5 Thermocouple, J6 ICSP, J9 RLY+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

Commit message: Add files via upload
Parts:
- moved C5 0.13 mm to (19.0, 38.3)
- moved C7 0.13 mm to (19.0, 41.7)
Routing:
- net GND: track 17.0 -> 18.7 mm
Changed lines of the file:
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@@
 <?xml version="1.0" encoding="utf-8"?>
 <!DOCTYPE eagle SYSTEM "eagle.dtd">
-<eagle version="8.3.2">
+<eagle version="8.4.0">
 <drawing>
 <settings>
@@
 <setting verticaltext="up"/>
 </settings>
-<grid distance="50" unitdist="mil" unit="mil" style="lines" multiple="1" display="yes" altdistance="25" altunitdist="mil" altunit="mil"/>
+<grid distance="50" unitdist="mil" unit="mil" style="lines" multiple="1" display="yes" altdistance="5" altunitdist="mil" altunit="mil"/>
 <layers>
 <layer number="1" name="Top" color="4" fill="1" visible="yes" active="yes"/>
@@
 <layer number="23" name="tOrigins" color="15" fill="1" visible="yes" active="yes"/>
 <layer number="24" name="bOrigins" color="15" fill="1" visible="yes" active="yes"/>
-<layer number="25" name="tNames" color="7" fill="1" visible="yes" active="yes"/>
+<layer number="25" name="tNames" color="7" fill="1" visible="no" active="yes"/>
 <layer number="26" name="bNames" color="7" fill="1" visible="no" active="yes"/>
 <layer number="27" name="tValues" color="7" fill="1" visible="no" active="yes"/>
@@
 <param name="dpMaxLengthDifference" value="10mm"/>
 <param name="dpGapFactor" value="2.5"/>
-<param name="checkGrid" value="0"/>
-<param name="checkAngle" value="1"/>
 <param name="checkFont" value="1"/>
 <param name="checkRestrict" value="1"/>
+<param name="checkStop" value="0"/>
 <param name="useDiameter" value="13"/>
 <param name="maxErrors" value="50"/>
@@
 <attribute name="VALUE" x="44.087696875" y="7.0124" size="0.8128" layer="27" font="vector" ratio="16"/>
 </element>
-<element name="C7" library="TimWoo-Capacitors" library_urn="urn:adsk.eagle:library:500759" package="0603-CAP-MARKED" package3d_urn="urn:adsk.eagle:package:500792/2" value="1uF" x="18.8595" y="41.656" smashed="yes" rot="R270">
-<attribute name="NAME" x="18.542" y="43.434" size="0.8128" layer="25" font="vector" ratio="16"/>
-<attribute name="VALUE" x="17.7165" y="42.672" size="0.8128" layer="27" font="vector" ratio="16" rot="R270"/>
+<element name="C7" library="TimWoo-Capacitors" library_urn="urn:adsk.eagle:library:500759" package="0603-CAP-MARKED" package3d_urn="urn:adsk.eagle:package:500792/2" value="1uF" x="18.9865" y="41.656" smashed="yes" rot="R270">
+<attribute name="NAME" x="18.669" y="43.434" size="0.8128" layer="25" font="vector" ratio="16"/>
+<attribute name="VALUE" x="17.8435" y="42.672" size="0.8128" layer="27" font="vector" ratio="16" rot="R270"/>
 </element>
 <element name="C2" library="TimWoo-Capacitors" library_urn="urn:adsk.eagle:library:500759" package="0603-CAP-MARKED" package3d_urn="urn:adsk.eagle:package:500792/2" value="0.1uF" x="32.1671" y="23.513696875" smashed="yes" rot="R90">
@@
 <attribute name="VALUE" x="12.954" y="39.5605" size="0.8128" layer="27" font="vector" ratio="16" rot="R180"/>
 </element>
-<element name="C5" library="TimWoo-Capacitors" library_urn="urn:adsk.eagle:library:500759" package="0603-CAP-MARKED" package3d_urn="urn:adsk.eagle:package:500792/2" value="4.7uF" x="18.8595" y="38.2905" smashed="yes" rot="R90">
-<attribute name="NAME" x="19.7485" y="38.862" size="0.8128" layer="25" font="vector" ratio="16" rot="R270"/>
-<attribute name="VALUE" x="20.0025" y="37.2745" size="0.8128" layer="27" font="vector" ratio="16" rot="R90"/>
+<element name="C5" library="TimWoo-Capacitors" library_urn="urn:adsk.eagle:library:500759" package="0603-CAP-MARKED" package3d_urn="urn:adsk.eagle:package:500792/2" value="4.7uF" x="18.9865" y="38.2905" smashed="yes" rot="R90">
+<attribute name="NAME" x="19.8755" y="38.862" size="0.8128" layer="25" font="vector" ratio="16" rot="R270"/>
+<attribute name="VALUE" x="20.1295" y="37.2745" size="0.8128" layer="27" font="vector" ratio="16" rot="R90"/>
 </element>
 <element name="J2" library="TimWoo-Connectors" package="JST-2-SMD" value="LiPo Battery" x="11.7475" y="3.81" smashed="yes" rot="R180">
@@
 <contactref element="D3" pad="C"/>
 <contactref element="D5" pad="C"/>
-<polygon width="0.1524" layer="1">
+<polygon width="0.3048" layer="1">
 <vertex x="-1.27" y="54.61"/>
 <vertex x="58.42" y="54.61"/>
@@
 <wire x1="17.1751" y1="35.687" x2="17.907" y2="35.687" width="0.6096" layer="1"/>
 <wire x1="17.907" y1="35.687" x2="18.161" y2="35.433" width="0.6096" layer="1"/>
-<wire x1="14.5749" y1="41.656" x2="15.748" y2="41.656" width="0.6096" layer="1"/>
+<wire x1="15.748" y1="41.656" x2="14.5749" y2="41.656" width="0.6096" layer="1"/>
 <via x="17.78" y="7.62" extent="1-16" drill="0.508" diameter="1.016"/>
 <via x="14.478" y="43.815" extent="1-16" drill="0.508" diameter="1.016"/>
@@
 <via x="45.085" y="10.795" extent="1-16" drill="0.508" diameter="1.016"/>
 <contactref element="IC2" pad="33"/>
+<wire x1="18.9865" y1="39.1405" x2="18.9865" y2="39.878" width="0.8128" layer="1"/>
+<wire x1="18.9865" y1="39.878" x2="18.034" y2="39.878" width="0.8128" layer="1"/>
 </signal>
 <signal name="V_USB" class="1">
@@
 <wire x1="35.37" y1="8.7625" x2="35.56" y2="8.5725" width="0.4064" layer="1"/>
 <wire x1="35.56" y1="8.5725" x2="35.56" y2="7.0739" width="0.4064" layer="1"/>
-<wire x1="18.8595" y1="42.506" x2="19.597" y2="42.506" width="0.508" layer="1"/>
+<wire x1="18.9865" y1="42.506" x2="19.597" y2="42.506" width="0.508" layer="1"/>
 <wire x1="19.597" y1="42.506" x2="20.193" y2="41.91" width="0.508" layer="1"/>
 <wire x1="20.193" y1="41.91" x2="20.193" y2="36.957" width="0.508" layer="1"/>
 <wire x1="20.193" y1="36.957" x2="20.955" y2="36.195" width="0.508" layer="1"/>
 <wire x1="17.1751" y1="42.606" x2="18.7595" y2="42.606" width="0.508" layer="1"/>
-<wire x1="18.7595" y1="42.606" x2="18.8595" y2="42.506" width="0.508" layer="1"/>
+<wire x1="18.7595" y1="42.606" x2="18.9865" y2="42.506" width="0.508" layer="1"/>
 <wire x1="25.5025" y1="13.8675" x2="26.3525" y2="13.8675" width="0.4064" layer="1"/>
 <wire x1="25.1345" y1="14.2355" x2="24.4475" y2="14.2355" width="0.4064" layer="1"/>
@@
 <wire x1="11.1125" y1="22.5425" x2="11.1125" y2="19.05" width="0.508" layer="1"/>
 <via x="11.1125" y="19.05" extent="1-16" drill="0.508" diameter="1.016"/>
-<via x="18.8595" y="36.195" extent="1-16" drill="0.508" diameter="1.016"/>
-<wire x1="17.78" y1="25.7175" x2="17.78" y2="35.1155" width="0.508" layer="16"/>
+<via x="18.9865" y="36.068" extent="1-16" drill="0.508" diameter="1.016"/>
+<wire x1="17.78" y1="25.7175" x2="17.78" y2="34.9885" width="0.508" layer="16"/>
 <wire x1="17.1751" y1="37.3681" x2="17.1751" y2="36.637" width="0.508" layer="1"/>
 <wire x1="17.35" y1="37.543" x2="17.35" y2="38.6715" width="0.508" layer="1"/>
 <wire x1="17.2475" y1="37.4405" x2="17.35" y2="37.543" width="0.508" layer="1"/>
-<wire x1="18.8595" y1="36.195" x2="18.8595" y2="37.4405" width="0.508" layer="1"/>
-<wire x1="17.78" y1="35.1155" x2="18.8595" y2="36.195" width="0.508" layer="16"/>
-<wire x1="18.8595" y1="37.4405" x2="17.2475" y2="37.4405" width="0.508" layer="1"/>
+<wire x1="18.9865" y1="36.068" x2="18.9865" y2="37.4405" width="0.508" layer="1"/>
+<wire x1="17.78" y1="34.9885" x2="18.9865" y2="36.068" width="0.508" layer="16"/>
+<wire x1="18.9865" y1="37.4405" x2="17.2475" y2="37.4405" width="0.508" layer="1"/>
 <wire x1="17.2475" y1="37.4405" x2="17.1751" y2="37.3681" width="0.508" layer="1"/>
 <wire x1="12.7635" y1="24.1935" x2="16.256" y2="24.1935" width="0.508" layer="16"/>

Commit message: Add files via upload
Parts:
- J1: device TimWoo-Connectors:USB-B-MICRO-SMD-V2 -> TimWoo-Connectors:USB-B-MICRO-SMD
Routing:
- net GND: track 18.7 -> 19.9 mm
Changed lines of the file:
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@@
 <attribute name="VALUE" x="20.8915" y="16.7005" size="0.8128" layer="27" ratio="13"/>
 </element>
-<element name="J1" library="TimWoo-Connectors" library_urn="urn:adsk.eagle:library:500889" package="USB-B-MICRO-SMD-V2" package3d_urn="urn:adsk.eagle:package:501328/2" value="microUSB" x="2.032" y="37.7825" smashed="yes">
+<element name="J1" library="TimWoo-Connectors" library_urn="urn:adsk.eagle:library:500889" package="USB-B-MICRO-SMD" package3d_urn="urn:adsk.eagle:package:501330/2" value="microUSB" x="2.032" y="37.7825" smashed="yes">
 <attribute name="NAME" x="0.762" y="35.4965" size="0.8128" layer="25" font="vector" ratio="16"/>
 <attribute name="VALUE" x="0.762" y="43.2435" size="0.8128" layer="27"/>
@@
 <contactref element="R6" pad="1"/>
 <contactref element="JP1" pad="1"/>
-<wire x1="4.757" y1="36.4825" x2="6.0025" y2="36.4825" width="0.4064" layer="1"/>
+<wire x1="6.0025" y1="36.4825" x2="4.757" y2="36.4825" width="0.4064" layer="1"/>
 <wire x1="6.0025" y1="36.4825" x2="6.0325" y2="36.5125" width="0.4064" layer="1"/>
 <wire x1="30.48" y1="3.683" x2="30.48" y2="2.54" width="0.8128" layer="1"/>
@@
 <wire x1="18.9865" y1="39.1405" x2="18.9865" y2="39.878" width="0.8128" layer="1"/>
 <wire x1="18.9865" y1="39.878" x2="18.034" y2="39.878" width="0.8128" layer="1"/>
+<wire x1="4.757" y1="36.4825" x2="3.6495" y2="36.4825" width="0.4064" layer="1"/>
+<wire x1="3.6495" y1="36.4825" x2="3.556" y2="36.576" width="0.4064" layer="1"/>
 </signal>
 <signal name="V_USB" class="1">

Commit message: Add files via upload
Parts:
- added LOGO1: OSHW-LOGOL, SparkFun-Aesthetics:OSHW-LOGO-L
Other:
- board text added: "13"
- board text removed: "IO"
Changed lines of the file:
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@@
 <?xml version="1.0" encoding="utf-8"?>
 <!DOCTYPE eagle SYSTEM "eagle.dtd">
-<eagle version="8.4.0">
+<eagle version="8.4.1">
 <drawing>
 <settings>
@@
 <text x="52.705" y="49.022" size="1.27" layer="21" font="vector" ratio="16" rot="R270">0</text>
 <text x="0.3175" y="43.4975" size="0.8128" layer="21" font="vector" ratio="16">ON</text>
-<text x="0.4445" y="31.4325" size="0.8128" layer="21" font="vector" ratio="16">IO</text>
+<text x="0.4445" y="31.4325" size="0.8128" layer="21" font="vector" ratio="16">13</text>
 <text x="29.5275" y="28.2575" size="1.778" layer="21" font="vector" ratio="16" align="center">botletics.com</text>
 <polygon width="0.3048" layer="21">
@@
 <param name="dpMaxLengthDifference" value="10mm"/>
 <param name="dpGapFactor" value="2.5"/>
+<param name="checkAngle" value="0"/>
 <param name="checkFont" value="1"/>
 <param name="checkRestrict" value="1"/>
@@
 <attribute name="VALUE" x="48.26" y="8.128" size="0.4064" layer="27" font="vector" ratio="16"/>
 </element>
+<element name="LOGO1" library="SparkFun-Aesthetics" library_urn="urn:adsk.eagle:library:507" package="OSHW-LOGO-L" package3d_urn="urn:adsk.eagle:package:37097/1" value="OSHW-LOGOL" x="40.64" y="38.1" rot="MR0"/>
 </elements>
 <signals>

Commit message: Add files via upload
Parts:
- removed D4: MBR120, TimWoo-Diodes:SOD-123FL
- added LED1: Green, TimWoo-LED:LED-0603-MARKED
- D1: value Green -> MBR120; device TimWoo-LED:LED-0603-MARKED -> TimWoo-Diodes:SOD-123FL
- moved D1 13.4 mm to (15.9, 38.7), turned to 0 degrees
- renumbered D2 to LED2, D3 to LED3, D5 to LED4
Connections:
- net GND: now also LED1.C; no longer D1.C
- net N$9: now also LED1.A; no longer D1.A
- net VBAT: now also D1.A; no longer D4.A
- net V_USB: now also D1.C; no longer D4.C
Changed lines of the file:
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@@
 <layer number="14" name="Route14" color="1" fill="6" visible="no" active="no"/>
 <layer number="15" name="Route15" color="4" fill="6" visible="no" active="no"/>
-<layer number="16" name="Bottom" color="1" fill="1" visible="yes" active="yes"/>
+<layer number="16" name="Bottom" color="1" fill="1" visible="no" active="yes"/>
 <layer number="17" name="Pads" color="2" fill="1" visible="yes" active="yes"/>
 <layer number="18" name="Vias" color="2" fill="1" visible="yes" active="yes"/>
@@
 <layer number="20" name="Dimension" color="24" fill="1" visible="yes" active="yes"/>
 <layer number="21" name="tPlace" color="16" fill="1" visible="yes" active="yes"/>
-<layer number="22" name="bPlace" color="6" fill="1" visible="yes" active="yes"/>
+<layer number="22" name="bPlace" color="6" fill="1" visible="no" active="yes"/>
 <layer number="23" name="tOrigins" color="15" fill="1" visible="yes" active="yes"/>
 <layer number="24" name="bOrigins" color="15" fill="1" visible="yes" active="yes"/>
-<layer number="25" name="tNames" color="7" fill="1" visible="no" active="yes"/>
+<layer number="25" name="tNames" color="7" fill="1" visible="yes" active="yes"/>
 <layer number="26" name="bNames" color="7" fill="1" visible="no" active="yes"/>
 <layer number="27" name="tValues" color="7" fill="1" visible="no" active="yes"/>
@@
 <attribute name="VALUE" x="23.75164375" y="11.2023" size="0.8128" layer="27" font="vector" ratio="16" rot="R135"/>
 </element>
-<element name="D1" library="TimWoo-LED" library_urn="urn:adsk.eagle:library:501982" package="LED-0603-MARKED" package3d_urn="urn:adsk.eagle:package:502010/2" value="Green" x="3.4925" y="43.815" smashed="yes" rot="R180">
-<attribute name="NAME" x="4.5085" y="42.799" size="0.8128" layer="25" font="vector" ratio="16" rot="R180"/>
+<element name="LED1" library="TimWoo-LED" library_urn="urn:adsk.eagle:library:501982" package="LED-0603-MARKED" package3d_urn="urn:adsk.eagle:package:502010/2" value="Green" x="3.4925" y="43.815" smashed="yes" rot="R180">
+<attribute name="NAME" x="4.7625" y="42.926" size="0.8128" layer="25" font="vector" ratio="16" rot="R180"/>
 <attribute name="VALUE" x="4.5085" y="45.212" size="0.8128" layer="27" rot="R180"/>
 </element>
-<element name="D3" library="TimWoo-LED" library_urn="urn:adsk.eagle:library:501982" package="LED-0603-MARKED" package3d_urn="urn:adsk.eagle:package:502010/2" value="Red" x="3.4925" y="31.75" smashed="yes" rot="R180">
-<attribute name="NAME" x="3.302" y="32.512" size="0.8128" layer="25" font="vector" ratio="16"/>
+<element name="LED3" library="TimWoo-LED" library_urn="urn:adsk.eagle:library:501982" package="LED-0603-MARKED" package3d_urn="urn:adsk.eagle:package:502010/2" value="Red" x="3.4925" y="31.75" smashed="yes" rot="R180">
+<attribute name="NAME" x="4.572" y="30.861" size="0.8128" layer="25" font="vector" ratio="16" rot="R180"/>
 <attribute name="VALUE" x="4.5085" y="33.147" size="0.8128" layer="27" rot="R180"/>
 </element>
@@
 <attribute name="VALUE" x="18.415" y="30.226" size="0.8128" layer="27" font="vector" ratio="16"/>
 </element>
-<element name="D5" library="TimWoo-LED" library_urn="urn:adsk.eagle:library:501982" package="LED-0603-MARKED" package3d_urn="urn:adsk.eagle:package:502010/2" value="Blue" x="20.828" y="27.8765" smashed="yes" rot="R270">
-<attribute name="NAME" x="21.717" y="27.178" size="0.8128" layer="25" font="vector" ratio="16" rot="R270"/>
+<element name="LED4" library="TimWoo-LED" library_urn="urn:adsk.eagle:library:501982" package="LED-0603-MARKED" package3d_urn="urn:adsk.eagle:package:502010/2" value="Blue" x="20.828" y="27.8765" smashed="yes" rot="R270">
+<attribute name="NAME" x="21.717" y="26.289" size="0.8128" layer="25" font="vector" ratio="16"/>
 <attribute name="VALUE" x="19.431" y="28.8925" size="0.8128" layer="27" rot="R270"/>
 </element>
@@
 <attribute name="VALUE" x="13.0175" y="3.81" size="0.8128" layer="27" rot="R180"/>
 </element>
-<element name="D2" library="TimWoo-LED" library_urn="urn:adsk.eagle:library:501982" package="LED-0603-MARKED" package3d_urn="urn:adsk.eagle:package:502010/2" value="Green" x="15.875" y="33.147" smashed="yes" rot="R180">
-<attribute name="NAME" x="15.367" y="33.9725" size="0.8128" layer="25" font="vector" ratio="16"/>
+<element name="LED2" library="TimWoo-LED" library_urn="urn:adsk.eagle:library:501982" package="LED-0603-MARKED" package3d_urn="urn:adsk.eagle:package:502010/2" value="Green" x="15.875" y="33.147" smashed="yes" rot="R180">
+<attribute name="NAME" x="14.605" y="30.4165" size="0.8128" layer="25" font="vector" ratio="16"/>
 <attribute name="VALUE" x="16.891" y="34.544" size="0.8128" layer="27" rot="R180"/>
 </element>
@@
 <attribute name="VALUE" x="10.7315" y="31.75" size="0.8128" layer="27" font="vector" ratio="16" align="top-center"/>
 </element>
-<element name="D4" library="TimWoo-Diodes" library_urn="urn:adsk.eagle:library:501758" package="SOD-123FL" package3d_urn="urn:adsk.eagle:package:501788/2" value="MBR120" x="15.875" y="38.6715" smashed="yes">
+<element name="D1" library="TimWoo-Diodes" library_urn="urn:adsk.eagle:library:501758" package="SOD-123FL" package3d_urn="urn:adsk.eagle:package:501788/2" value="MBR120" x="15.875" y="38.6715" smashed="yes">
 <attribute name="NAME" x="18.2245" y="39.243" size="0.8128" layer="25" font="vector" ratio="16" rot="R270"/>
 <attribute name="VALUE" x="14.859" y="37.2745" size="0.8128" layer="27"/>
@@
 <contactref element="IC4" pad="1"/>
 <contactref element="C8" pad="2"/>
-<contactref element="D1" pad="C"/>
+<contactref element="LED1" pad="C"/>
 <contactref element="J6" pad="6"/>
-<contactref element="D3" pad="C"/>
-<contactref element="D5" pad="C"/>
+<contactref element="LED3" pad="C"/>
+<contactref element="LED4" pad="C"/>
 <polygon width="0.3048" layer="1">
 <vertex x="-1.27" y="54.61"/>
@@
 <contactref element="IC1" pad="2"/>
 <contactref element="J2" pad="1"/>
-<contactref element="D2" pad="C"/>
+<contactref element="LED2" pad="C"/>
 <contactref element="R6" pad="1"/>
 <contactref element="JP1" pad="1"/>
@@
 <contactref element="IC3" pad="1"/>
 <contactref element="IC3" pad="3"/>
-<contactref element="D4" pad="C"/>
+<contactref element="D1" pad="C"/>
 <via x="13.0175" y="41.021" extent="1-16" drill="0.508" diameter="1.016"/>
 <contactref element="JP3" pad="1"/>
@@
 <signal name="N$9">
 <contactref element="R1" pad="2"/>
-<contactref element="D1" pad="A"/>
+<contactref element="LED1" pad="A"/>
 <wire x1="4.3695" y1="43.815" x2="6.135" y2="43.815" width="0.3048" layer="1"/>
 </signal>
@@
 <signal name="N$31">
 <contactref element="R8" pad="2"/>
-<contactref element="D3" pad="A"/>
+<contactref element="LED3" pad="A"/>
 <wire x1="4.3695" y1="31.75" x2="6.135" y2="31.75" width="0.3048" layer="1"/>
 </signal>
@@
 <contactref element="C5" pad="1"/>
 <contactref element="J2" pad="2"/>
-<contactref element="D4" pad="A"/>
+<contactref element="D1" pad="A"/>
 <contactref element="IC1" pad="3"/>
 <via x="11.1125" y="12.0015" extent="1-16" drill="0.508" diameter="1.016"/>
@@
 </signal>
 <signal name="N$6">
-<contactref element="D2" pad="A"/>
+<contactref element="LED2" pad="A"/>
 <contactref element="R3" pad="2"/>
 <wire x1="16.752" y1="33.147" x2="18.581" y2="33.147" width="0.3048" layer="1"/>
@@
 <signal name="N$11">
 <contactref element="R11" pad="2"/>
-<contactref element="D5" pad="A"/>
+<contactref element="LED4" pad="A"/>
 <wire x1="20.828" y1="28.7535" x2="20.828" y2="29.845" width="0.3048" layer="1"/>
 <wire x1="20.281" y1="30.392" x2="20.281" y2="31.369" width="0.3048" layer="1"/>
