File: PCB Files/Reflowduino Pro/Reflowduino Pro v2.sch (EAGLE design)
At the start: 57 parts, among them IC1 MCP73831, IC2 ATMEGA32U4, IC3 AP2112K-3.3TRG1, IC4 MAX31855, J1 microUSB, J10 RLY-, J2 LiPo Battery, J5 Thermocouple, J6 ICSP, J9 RLY+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

Commit message: Add files via upload
Other:
- note added: "GPL-3.0"
Changed lines of the file:
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@@
 disable buzzer</text>
 <text x="132.08" y="215.9" size="1.778" layer="97">USB boot enable</text>
+<text x="401.828" y="16.764" size="3.81" layer="97">GPL-3.0</text>
 </plain>
 <instances>

Commit message: Add files via upload
Other:
- note added: "CC-BY-SA-4.0"
- note removed: "GPL-3.0"
Changed lines of the file:
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@@
 disable buzzer</text>
 <text x="132.08" y="215.9" size="1.778" layer="97">USB boot enable</text>
-<text x="401.828" y="16.764" size="3.81" layer="97">GPL-3.0</text>
+<text x="399.288" y="24.384" size="3.81" layer="97">CC-BY-SA-4.0</text>
 </plain>
 <instances>

Commit message: Add files via upload
Parts:
- J1: device TimWoo-Connectors:MICRO-USB_SMD_NOSHIELDV2 -> TimWoo-Connectors:MICRO-USB_SMD_NOSHIELDV1
Changed lines of the file:
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@@
 <?xml version="1.0" encoding="utf-8"?>
 <!DOCTYPE eagle SYSTEM "eagle.dtd">
-<eagle version="8.3.2">
+<eagle version="8.4.0">
 <drawing>
 <settings>
@@
 <part name="GND26" library="TimWoo-Aesthetics" library_urn="urn:adsk.eagle:library:502097" deviceset="GND" device=""/>
 <part name="IC2" library="TimWoo-IC" library_urn="urn:adsk.eagle:library:500796" deviceset="ATMEGA32U4" device="-AU" package3d_urn="urn:adsk.eagle:package:500858/2" value="ATMEGA32U4"/>
-<part name="J1" library="TimWoo-Connectors" library_urn="urn:adsk.eagle:library:500889" deviceset="MICRO-USB_SMD_NOSHIELD" device="V2" package3d_urn="urn:adsk.eagle:package:501328/2" value="microUSB"/>
+<part name="J1" library="TimWoo-Connectors" library_urn="urn:adsk.eagle:library:500889" deviceset="MICRO-USB_SMD_NOSHIELD" device="V1" package3d_urn="urn:adsk.eagle:package:501330/2" value="microUSB"/>
 <part name="SUPPLY4" library="TimWoo-Aesthetics" library_urn="urn:adsk.eagle:library:502097" deviceset="V_USB" device=""/>
 <part name="IC3" library="TimWoo-IC" library_urn="urn:adsk.eagle:library:500796" deviceset="VOLTAGE-REGULATOR_SOT23-5" device="SOT-23-5" package3d_urn="urn:adsk.eagle:package:500846/2" value="AP2112K-3.3TRG1"/>

Commit message: Add files via upload
Parts:
- added LOGO1: OSHW-LOGOL, SparkFun-Aesthetics:OSHW-LOGOL
Changed lines of the file:
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@@
 <?xml version="1.0" encoding="utf-8"?>
 <!DOCTYPE eagle SYSTEM "eagle.dtd">
-<eagle version="8.4.0">
+<eagle version="8.4.1">
 <drawing>
 <settings>
@@
 <part name="R10" library="TimWoo-Resistors" library_urn="urn:adsk.eagle:library:500711" deviceset="RESISTOR" device="MARKED-0603" package3d_urn="urn:adsk.eagle:package:500751/2" value="10k"/>
 <part name="GND15" library="TimWoo-Aesthetics" library_urn="urn:adsk.eagle:library:502097" deviceset="GND" device=""/>
+<part name="LOGO1" library="SparkFun-Aesthetics" library_urn="urn:adsk.eagle:library:507" deviceset="OSHW-LOGO" device="L" package3d_urn="urn:adsk.eagle:package:37097/1" value="OSHW-LOGOL"/>
 </parts>
 <sheets>
@@
 <instance part="R10" gate="G$1" x="363.22" y="50.8"/>
 <instance part="GND15" gate="1" x="139.7" y="210.82" rot="R90"/>
+<instance part="LOGO1" gate="G$1" x="317.5" y="10.16"/>
 </instances>
 <busses>

Commit message: Add files via upload
Parts:
- removed D4: MBR120, TimWoo-Diodes:DIODE-SCHOTTKYSOD-123FL
- added LED1: Green, TimWoo-LED:LED0603-MARKED
- D1: value Green -> MBR120; device TimWoo-LED:LED0603-MARKED -> TimWoo-Diodes:DIODE-SCHOTTKYSOD-123FL
- renumbered D2 to LED2, D3 to LED3, D5 to LED4
Connections:
- net GND: now also LED1.C; no longer D1.C
- net N$9: now also LED1.A; no longer D1.A
- net VBAT: now also D1.A; no longer D4.A
- net V_USB: now also D1.C; no longer D4.C
Changed lines of the file:
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@@
 <part name="SUPPLY16" library="TimWoo-Aesthetics" library_urn="urn:adsk.eagle:library:502097" deviceset="3.3V" device=""/>
 <part name="GND22" library="TimWoo-Aesthetics" library_urn="urn:adsk.eagle:library:502097" deviceset="GND" device=""/>
-<part name="D1" library="TimWoo-LED" library_urn="urn:adsk.eagle:library:501982" deviceset="LED" device="0603-MARKED" package3d_urn="urn:adsk.eagle:package:502010/2" value="Green"/>
-<part name="D3" library="TimWoo-LED" library_urn="urn:adsk.eagle:library:501982" deviceset="LED" device="0603-MARKED" package3d_urn="urn:adsk.eagle:package:502010/2" value="Red"/>
+<part name="LED1" library="TimWoo-LED" library_urn="urn:adsk.eagle:library:501982" deviceset="LED" device="0603-MARKED" package3d_urn="urn:adsk.eagle:package:502010/2" value="Green"/>
+<part name="LED3" library="TimWoo-LED" library_urn="urn:adsk.eagle:library:501982" deviceset="LED" device="0603-MARKED" package3d_urn="urn:adsk.eagle:package:502010/2" value="Red"/>
 <part name="R1" library="TimWoo-Resistors" library_urn="urn:adsk.eagle:library:500711" deviceset="RESISTOR" device="MARKED-0603" package3d_urn="urn:adsk.eagle:package:500751/2" value="2k"/>
 <part name="R8" library="TimWoo-Resistors" library_urn="urn:adsk.eagle:library:500711" deviceset="RESISTOR" device="MARKED-0603" package3d_urn="urn:adsk.eagle:package:500751/2" value="470"/>
@@
 <part name="U1" library="TimWoo-RF" library_urn="urn:adsk.eagle:library:527286" deviceset="HM-11_JDY-08_BLUETOOTH" device="" value="HM-11 Bluetooth"/>
 <part name="R11" library="TimWoo-Resistors" library_urn="urn:adsk.eagle:library:500711" deviceset="RESISTOR" device="MARKED-0603" package3d_urn="urn:adsk.eagle:package:500751/2" value="470"/>
-<part name="D5" library="TimWoo-LED" library_urn="urn:adsk.eagle:library:501982" deviceset="LED" device="0603-MARKED" package3d_urn="urn:adsk.eagle:package:502010/2" value="Blue"/>
+<part name="LED4" library="TimWoo-LED" library_urn="urn:adsk.eagle:library:501982" deviceset="LED" device="0603-MARKED" package3d_urn="urn:adsk.eagle:package:502010/2" value="Blue"/>
 <part name="GND29" library="TimWoo-Aesthetics" library_urn="urn:adsk.eagle:library:502097" deviceset="GND" device=""/>
 <part name="GND28" library="TimWoo-Aesthetics" library_urn="urn:adsk.eagle:library:502097" deviceset="GND" device=""/>
@@
 <part name="C5" library="TimWoo-Capacitors" library_urn="urn:adsk.eagle:library:500759" deviceset="CAP" device="MARKED-0603" package3d_urn="urn:adsk.eagle:package:500792/2" value="4.7uF"/>
 <part name="J2" library="TimWoo-Connectors" deviceset="M02" device="-JST-2MM-SMT" value="LiPo Battery"/>
-<part name="D2" library="TimWoo-LED" library_urn="urn:adsk.eagle:library:501982" deviceset="LED" device="0603-MARKED" package3d_urn="urn:adsk.eagle:package:502010/2" value="Green"/>
+<part name="LED2" library="TimWoo-LED" library_urn="urn:adsk.eagle:library:501982" deviceset="LED" device="0603-MARKED" package3d_urn="urn:adsk.eagle:package:502010/2" value="Green"/>
 <part name="GND8" library="SparkFun" deviceset="GND" device=""/>
 <part name="R3" library="TimWoo-Resistors" library_urn="urn:adsk.eagle:library:500711" deviceset="RESISTOR" device="MARKED-0603" package3d_urn="urn:adsk.eagle:package:500751/2" value="2k"/>
@@
 <part name="R7" library="TimWoo-Resistors" library_urn="urn:adsk.eagle:library:500711" deviceset="RESISTOR" device="MARKED-0603" package3d_urn="urn:adsk.eagle:package:500751/2" value="4.02k"/>
 <part name="JP1" library="TimWoo-Connectors" deviceset="JUMPER-SMT_2_NO" device="_SILK" value="500mA"/>
-<part name="D4" library="TimWoo-Diodes" library_urn="urn:adsk.eagle:library:501758" deviceset="DIODE-SCHOTTKY" device="SOD-123FL" package3d_urn="urn:adsk.eagle:package:501788/2" value="MBR120"/>
+<part name="D1" library="TimWoo-Diodes" library_urn="urn:adsk.eagle:library:501758" deviceset="DIODE-SCHOTTKY" device="SOD-123FL" package3d_urn="urn:adsk.eagle:package:501788/2" value="MBR120"/>
 <part name="SUPPLY8" library="TimWoo-Aesthetics" library_urn="urn:adsk.eagle:library:502097" deviceset="VBAT" device=""/>
 <part name="SUPPLY10" library="TimWoo-Aesthetics" library_urn="urn:adsk.eagle:library:502097" deviceset="VBAT" device=""/>
@@
 <instance part="SUPPLY16" gate="G$1" x="271.78" y="78.74"/>
 <instance part="GND22" gate="1" x="271.78" y="63.5"/>
-<instance part="D1" gate="G$1" x="17.78" y="142.24"/>
-<instance part="D3" gate="G$1" x="157.48" y="200.66" rot="R90"/>
+<instance part="LED1" gate="G$1" x="17.78" y="142.24"/>
+<instance part="LED3" gate="G$1" x="157.48" y="200.66" rot="R90"/>
 <instance part="R1" gate="G$1" x="17.78" y="152.4" rot="R270"/>
 <instance part="R8" gate="G$1" x="147.32" y="200.66"/>
@@
 <instance part="U1" gate="G$1" x="381" y="228.6"/>
 <instance part="R11" gate="G$1" x="403.86" y="220.98"/>
-<instance part="D5" gate="G$1" x="411.48" y="215.9"/>
+<instance part="LED4" gate="G$1" x="411.48" y="215.9"/>
 <instance part="GND29" gate="1" x="411.48" y="205.74"/>
 <instance part="GND28" gate="1" x="411.48" y="238.76" rot="R90"/>
@@
 <instance part="C5" gate="G$1" x="101.6" y="48.26"/>
 <instance part="J2" gate="G$1" x="121.92" y="55.88" rot="R180"/>
-<instance part="D2" gate="G$1" x="43.18" y="43.18"/>
+<instance part="LED2" gate="G$1" x="43.18" y="43.18"/>
 <instance part="GND8" gate="1" x="43.18" y="33.02"/>
 <instance part="R3" gate="G$1" x="50.8" y="50.8" rot="MR0"/>
@@
 <instance part="R7" gate="G$1" x="93.98" y="40.64" rot="R90"/>
 <instance part="JP1" gate="G$1" x="93.98" y="27.94" rot="R90"/>
-<instance part="D4" gate="G$1" x="182.88" y="66.04" rot="R270"/>
+<instance part="D1" gate="G$1" x="182.88" y="66.04" rot="R270"/>
 <instance part="SUPPLY8" gate="G$1" x="101.6" y="60.96"/>
 <instance part="SUPPLY10" gate="G$1" x="182.88" y="71.12"/>
@@
 </segment>
 <segment>
-<pinref part="D1" gate="G$1" pin="C"/>
+<pinref part="LED1" gate="G$1" pin="C"/>
 <pinref part="GND1" gate="1" pin="GND"/>
 <wire x1="17.78" y1="137.16" x2="17.78" y2="134.62" width="0.1524" layer="91"/>
@@
 </segment>
 <segment>
-<pinref part="D3" gate="G$1" pin="C"/>
+<pinref part="LED3" gate="G$1" pin="C"/>
 <pinref part="GND16" gate="1" pin="GND"/>
 <wire x1="162.56" y1="200.66" x2="165.1" y2="200.66" width="0.1524" layer="91"/>
@@
 </segment>
 <segment>
-<pinref part="D5" gate="G$1" pin="C"/>
+<pinref part="LED4" gate="G$1" pin="C"/>
 <pinref part="GND29" gate="1" pin="GND"/>
 <wire x1="411.48" y1="210.82" x2="411.48" y2="208.28" width="0.1524" layer="91"/>
@@
 </segment>
 <segment>
-<pinref part="D2" gate="G$1" pin="C"/>
+<pinref part="LED2" gate="G$1" pin="C"/>
 <pinref part="GND8" gate="1" pin="GND"/>
 <wire x1="43.18" y1="38.1" x2="43.18" y2="35.56" width="0.1524" layer="91"/>
@@
 <wire x1="185.42" y1="53.34" x2="182.88" y2="53.34" width="0.1524" layer="91"/>
 <wire x1="182.88" y1="53.34" x2="182.88" y2="55.88" width="0.1524" layer="91"/>
-<pinref part="D4" gate="G$1" pin="C"/>
+<pinref part="D1" gate="G$1" pin="C"/>
 <wire x1="182.88" y1="63.5" x2="182.88" y2="55.88" width="0.1524" layer="91"/>
 <junction x="182.88" y="55.88"/>
@@
 <segment>
 <pinref part="R1" gate="G$1" pin="2"/>
-<pinref part="D1" gate="G$1" pin="A"/>
+<pinref part="LED1" gate="G$1" pin="A"/>
 <wire x1="17.78" y1="147.32" x2="17.78" y2="144.78" width="0.1524" layer="91"/>
 </segment>
@@
 <segment>
 <pinref part="R8" gate="G$1" pin="2"/>
-<pinref part="D3" gate="G$1" pin="A"/>
+<pinref part="LED3" gate="G$1" pin="A"/>
 <wire x1="152.4" y1="200.66" x2="154.94" y2="200.66" width="0.1524" layer="91"/>
 </segment>
@@
 <segment>
 <pinref part="SUPPLY10" gate="G$1" pin="VBAT"/>
-<pinref part="D4" gate="G$1" pin="A"/>
+<pinref part="D1" gate="G$1" pin="A"/>
 <wire x1="182.88" y1="71.12" x2="182.88" y2="68.58" width="0.1524" layer="91"/>
 </segment>
@@
 <net name="N$6" class="0">
 <segment>
-<pinref part="D2" gate="G$1" pin="A"/>
+<pinref part="LED2" gate="G$1" pin="A"/>
 <pinref part="R3" gate="G$1" pin="2"/>
 <wire x1="45.72" y1="50.8" x2="43.18" y2="50.8" width="0.1524" layer="91"/>
@@
 <segment>
 <pinref part="R11" gate="G$1" pin="2"/>
-<pinref part="D5" gate="G$1" pin="A"/>
+<pinref part="LED4" gate="G$1" pin="A"/>
 <wire x1="408.94" y1="220.98" x2="411.48" y2="220.98" width="0.1524" layer="91"/>
 <wire x1="411.48" y1="220.98" x2="411.48" y2="218.44" width="0.1524" layer="91"/>
