File: PCB Files/Reflowduino Pro/Reflowduino Pro v3.brd (EAGLE design)
At the start: 86.4 x 53.3 mm, 56 parts, among them IC1 MCP73831, IC2 ATMEGA32U4, IC3 AP2112K-3.3TRG1, IC4 MAX31855, J1 microUSB, J10 RLY-, J2 LiPo Battery, J5 Thermocouple, J6 ICSP, J9 RLY+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

Commit message: Add files via upload
Other:
- board text added: "Reflowduino v3 botletics.com"
- board text removed: "Reflowduino v2.1 botletics.com"
Changed lines of the file:
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@@
 <wire x1="85.36" y1="53.34" x2="1" y2="53.34" width="0" layer="20"/>
 <wire x1="1" y1="53.34" x2="0" y2="52.34" width="0" layer="20" curve="90"/>
-<text x="28.575" y="26.67" size="3.81" layer="22" font="vector" ratio="16" rot="MR180" align="center">Reflowduino v2.1
+<text x="28.575" y="26.67" size="3.81" layer="22" font="vector" ratio="16" rot="MR180" align="center">Reflowduino v3
 botletics.com</text>
 <hole x="5.08" y="50.8" drill="3.2"/>
