File: PCB Files/Reflowduino Pro/Reflowduino Pro v3.sch (EAGLE design)
At the start: 56 parts, among them IC1 MCP73831, IC2 ATMEGA32U4, IC3 AP2112K-3.3TRG1, IC4 MAX31855, J1 microUSB, J10 RLY-, J2 LiPo Battery, J5 Thermocouple, J6 ICSP, J9 RLY+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

Commit message: Add files via upload
Other:
- note added: "v3"
- note removed: "v2.1"
Changed lines of the file:
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@@
 <plain>
 <text x="351.028" y="13.208" size="3.81" layer="97" align="top-left">Timothy Woo</text>
-<text x="419.608" y="6.604" size="3.81" layer="97">v2.1</text>
+<text x="419.608" y="6.604" size="3.81" layer="97">v3</text>
 <wire x1="431.8" y1="114.3" x2="431.8" y2="111.76" width="0.3048" layer="94"/>
 <text x="229.87" y="205.74" size="1.27" layer="91">IOREF</text>
