File: PCB Files/Reflowduino Basic/Reflowduino Basic v2.brd (EAGLE design)
At the start: 58.4 x 53.3 mm, 54 parts, among them IC1 MCP73831, IC2 ATMEGA32U4, IC3 AP2112K-3.3TRG1, IC4 MAX31855, J1 microUSB, J10 RLY-, J2 LiPo Battery, J5 Thermocouple, J6 ICSP, J9 RLY+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

Commit message: Add files via upload
Parts:
- J1: device TimWoo-Connectors:USB-B-MICRO-SMD-V2 -> TimWoo-Connectors:USB-B-MICRO-SMD
Routing:
- net GND: track 20.3 -> 21.6 mm
Changed lines of the file:
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@@
 <attribute name="VALUE" x="20.8915" y="16.7005" size="0.8128" layer="27" ratio="13"/>
 </element>
-<element name="J1" library="TimWoo-Connectors" library_urn="urn:adsk.eagle:library:500889" package="USB-B-MICRO-SMD-V2" package3d_urn="urn:adsk.eagle:package:501328/2" value="microUSB" x="2.032" y="37.7825" smashed="yes">
+<element name="J1" library="TimWoo-Connectors" library_urn="urn:adsk.eagle:library:500889" package="USB-B-MICRO-SMD" package3d_urn="urn:adsk.eagle:package:501330/2" value="microUSB" x="2.032" y="37.7825" smashed="yes">
 <attribute name="NAME" x="0.762" y="35.4965" size="0.8128" layer="25" font="vector" ratio="16"/>
 <attribute name="VALUE" x="0.762" y="43.2435" size="0.8128" layer="27"/>
@@
 <contactref element="R6" pad="1"/>
 <contactref element="JP1" pad="1"/>
-<wire x1="4.757" y1="36.4825" x2="6.0025" y2="36.4825" width="0.4064" layer="1"/>
+<wire x1="6.0025" y1="36.4825" x2="4.757" y2="36.4825" width="0.4064" layer="1"/>
 <wire x1="6.0025" y1="36.4825" x2="6.0325" y2="36.5125" width="0.4064" layer="1"/>
 <wire x1="30.48" y1="3.683" x2="30.48" y2="2.54" width="0.8128" layer="1"/>
@@
 <wire x1="18.9865" y1="39.1405" x2="18.9865" y2="39.878" width="0.8128" layer="1"/>
 <wire x1="18.9865" y1="39.878" x2="18.034" y2="39.878" width="0.8128" layer="1"/>
+<wire x1="4.757" y1="36.4825" x2="3.5895" y2="36.4825" width="0.4064" layer="1"/>
+<wire x1="3.5895" y1="36.4825" x2="3.556" y2="36.449" width="0.4064" layer="1"/>
 </signal>
 <signal name="V_USB" class="1">

Commit message: Add files via upload
Parts:
- added LOGO1: OSHW-LOGOL, SparkFun-Aesthetics:OSHW-LOGO-L
Changed lines of the file:
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@@
 <?xml version="1.0" encoding="utf-8"?>
 <!DOCTYPE eagle SYSTEM "eagle.dtd">
-<eagle version="8.4.0">
+<eagle version="8.4.1">
 <drawing>
 <settings>
@@
 <param name="dpMaxLengthDifference" value="10mm"/>
 <param name="dpGapFactor" value="2.5"/>
+<param name="checkAngle" value="0"/>
 <param name="checkFont" value="1"/>
 <param name="checkRestrict" value="1"/>
@@
 <attribute name="VALUE" x="48.26" y="8.128" size="0.4064" layer="27" font="vector" ratio="16"/>
 </element>
+<element name="LOGO1" library="SparkFun-Aesthetics" library_urn="urn:adsk.eagle:library:507" package="OSHW-LOGO-L" package3d_urn="urn:adsk.eagle:package:37097/1" value="OSHW-LOGOL" x="40.64" y="38.1" rot="MR0"/>
 </elements>
 <signals>
