File: PCB Files/Reflowduino Basic/Reflowduino Basic v2.sch (EAGLE design)
At the start: 54 parts, among them IC1 MCP73831, IC2 ATMEGA32U4, IC3 AP2112K-3.3TRG1, IC4 MAX31855, J1 microUSB, J10 RLY-, J2 LiPo Battery, J5 Thermocouple, J6 ICSP, J9 RLY+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

Commit message: Add files via upload
Parts:
- J1: device TimWoo-Connectors:MICRO-USB_SMD_NOSHIELDV2 -> TimWoo-Connectors:MICRO-USB_SMD_NOSHIELDV1
Changed lines of the file:
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@@
 <part name="GND26" library="TimWoo-Aesthetics" library_urn="urn:adsk.eagle:library:502097" deviceset="GND" device=""/>
 <part name="IC2" library="TimWoo-IC" library_urn="urn:adsk.eagle:library:500796" deviceset="ATMEGA32U4" device="-AU" package3d_urn="urn:adsk.eagle:package:500858/2" value="ATMEGA32U4"/>
-<part name="J1" library="TimWoo-Connectors" library_urn="urn:adsk.eagle:library:500889" deviceset="MICRO-USB_SMD_NOSHIELD" device="V2" package3d_urn="urn:adsk.eagle:package:501328/2" value="microUSB"/>
+<part name="J1" library="TimWoo-Connectors" library_urn="urn:adsk.eagle:library:500889" deviceset="MICRO-USB_SMD_NOSHIELD" device="V1" package3d_urn="urn:adsk.eagle:package:501330/2" value="microUSB"/>
 <part name="SUPPLY4" library="TimWoo-Aesthetics" library_urn="urn:adsk.eagle:library:502097" deviceset="V_USB" device=""/>
 <part name="IC3" library="TimWoo-IC" library_urn="urn:adsk.eagle:library:500796" deviceset="VOLTAGE-REGULATOR_SOT23-5" device="SOT-23-5" package3d_urn="urn:adsk.eagle:package:500846/2" value="AP2112K-3.3TRG1"/>

Commit message: Add files via upload
Parts:
- added LOGO1: OSHW-LOGOL, SparkFun-Aesthetics:OSHW-LOGOL
Changed lines of the file:
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@@
 <?xml version="1.0" encoding="utf-8"?>
 <!DOCTYPE eagle SYSTEM "eagle.dtd">
-<eagle version="8.4.0">
+<eagle version="8.4.1">
 <drawing>
 <settings>
@@
 <part name="R10" library="TimWoo-Resistors" library_urn="urn:adsk.eagle:library:500711" deviceset="RESISTOR" device="MARKED-0603" package3d_urn="urn:adsk.eagle:package:500751/2" value="10k"/>
 <part name="GND15" library="TimWoo-Aesthetics" library_urn="urn:adsk.eagle:library:502097" deviceset="GND" device=""/>
+<part name="LOGO1" library="SparkFun-Aesthetics" library_urn="urn:adsk.eagle:library:507" deviceset="OSHW-LOGO" device="L" package3d_urn="urn:adsk.eagle:package:37097/1" value="OSHW-LOGOL"/>
 </parts>
 <sheets>
@@
 <instance part="R10" gate="G$1" x="363.22" y="50.8"/>
 <instance part="GND15" gate="1" x="139.7" y="210.82" rot="R90"/>
+<instance part="LOGO1" gate="G$1" x="317.5" y="10.16"/>
 </instances>
 <busses>
