File: PCB Files/Solid-State Sidekick/Solid-State Sidekick v1.brd (EAGLE design)
At the start: 66 x 72.4 mm, 5 parts, among them J1 C14, J2 NEMA, J3 RLY Control, SW1 Rocker

Commit message: Add files via upload
Parts:
- added LOGO1: OSHW-LOGOL, SparkFun-Aesthetics:OSHW-LOGO-L
Changed lines of the file:
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@@
 <element name="RLY1" library="TimWoo-Electromechanical" library_urn="urn:adsk.eagle:library:501864" package="RELAY_PF240" package3d_urn="urn:adsk.eagle:package:501907/3" value="PF240D25R" x="43.18" y="53.34"/>
 <element name="SW1" library="TimWoo-Electromechanical" library_urn="urn:adsk.eagle:library:501864" package="R1966ABLKBLKFR" value="Rocker" x="15.24" y="60.96" rot="R90"/>
+<element name="LOGO1" library="SparkFun-Aesthetics" library_urn="urn:adsk.eagle:library:507" package="OSHW-LOGO-L" package3d_urn="urn:adsk.eagle:package:37097/1" value="OSHW-LOGOL" x="54.61" y="5.08" rot="MR0"/>
 </elements>
 <signals>

Commit message: Add files via upload
Routing:
- net GND: track 27.9 -> 31.3 mm
- net L_SW: track 7.93 -> 9.67 mm
Changed lines of the file:
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@@
 <hole x="62.21" y="5.65" drill="3.5"/>
 <text x="48.895" y="67.31" size="1.27" layer="21" font="vector" ratio="16" rot="R90">RLY-</text>
-<text x="39.37" y="67.31" size="1.27" layer="21" font="vector" ratio="16" rot="R90">RLY+</text>
+<text x="39.116" y="67.31" size="1.27" layer="21" font="vector" ratio="16" rot="R90">RLY+</text>
 <text x="30.48" y="1.27" size="2.54" layer="21" font="vector" ratio="16">botletics.com</text>
 <text x="22.86" y="6.35" size="2.54" layer="21" font="vector" ratio="16">Solid-State Sidekick v1</text>
@@
 <contactref element="J1" pad="E"/>
 <contactref element="J2" pad="GND"/>
-<wire x1="16.51" y1="25.4" x2="44.45" y2="25.4" width="3.81" layer="1"/>
+<wire x1="16.51" y1="25.4" x2="47.83" y2="25.4" width="3.81" layer="1"/>
 </signal>
 <signal name="N">
@@
 <vertex x="12.065" y="26.67"/>
 <vertex x="12.065" y="21.59"/>
-<vertex x="48.895" y="21.59"/>
-<vertex x="48.895" y="26.67"/>
+<vertex x="52.07" y="21.59"/>
+<vertex x="52.07" y="26.67"/>
 <vertex x="64.77" y="26.67"/>
 <vertex x="64.77" y="1.27"/>
@@
 <vertex x="12.065" y="26.67"/>
 <vertex x="12.065" y="21.59"/>
-<vertex x="48.895" y="21.59"/>
-<vertex x="48.895" y="26.67"/>
+<vertex x="52.07" y="21.59"/>
+<vertex x="52.07" y="26.67"/>
 <vertex x="64.77" y="26.67"/>
 <vertex x="64.77" y="1.27"/>
@@
 <via x="54.61" y="24.13" extent="1-16" drill="0.635" diameter="1.27"/>
 <via x="60.96" y="24.13" extent="1-16" drill="0.635" diameter="1.27"/>
-<wire x1="40.26" y1="19.05" x2="40.64" y2="18.67" width="5.08" layer="1"/>
-<wire x1="40.64" y1="18.67" x2="40.64" y2="16.51" width="5.08" layer="1"/>
-<wire x1="40.26" y1="19.05" x2="40.64" y2="18.67" width="5.08" layer="16"/>
-<wire x1="40.64" y1="18.67" x2="40.64" y2="16.51" width="5.08" layer="16"/>
 <via x="35.56" y="17.78" extent="1-16" drill="0.635" diameter="1.27"/>
+<wire x1="43.64" y1="19.05" x2="43.64" y2="16.05" width="5.08" layer="1"/>
+<wire x1="43.64" y1="16.05" x2="43.815" y2="15.875" width="5.08" layer="1"/>
+<wire x1="43.64" y1="19.05" x2="43.64" y2="16.685" width="5.08" layer="16"/>
+<wire x1="43.64" y1="16.685" x2="43.815" y2="16.51" width="5.08" layer="16"/>
 </signal>
 <signal name="L_WALL">
@@
 <wire x1="39.37" y1="53.34" x2="41.91" y2="53.34" width="5.08" layer="1"/>
 <wire x1="39.37" y1="53.34" x2="41.91" y2="53.34" width="5.08" layer="16"/>
-<wire x1="40.26" y1="31.75" x2="40.26" y2="32.64" width="5.08" layer="16"/>
-<wire x1="40.26" y1="32.64" x2="40.64" y2="33.02" width="5.08" layer="16"/>
-<wire x1="40.26" y1="31.75" x2="40.26" y2="32.64" width="5.08" layer="1"/>
-<wire x1="40.26" y1="32.64" x2="40.64" y2="33.02" width="5.08" layer="1"/>
-<via x="44.45" y="30.48" extent="1-16" drill="0.635" diameter="1.27"/>
+<via x="38.1" y="30.48" extent="1-16" drill="0.635" diameter="1.27"/>
 <via x="57.15" y="49.53" extent="1-16" drill="0.635" diameter="1.27"/>
 <via x="63.5" y="49.53" extent="1-16" drill="0.635" diameter="1.27"/>
@@
 <via x="38.1" y="62.23" extent="1-16" drill="0.635" diameter="1.27"/>
 <via x="47.625" y="52.705" extent="1-16" drill="0.635" diameter="1.27"/>
+<wire x1="43.64" y1="31.75" x2="43.64" y2="34.115" width="5.08" layer="16"/>
+<wire x1="43.64" y1="34.115" x2="43.815" y2="34.29" width="5.08" layer="16"/>
+<wire x1="43.64" y1="31.75" x2="43.64" y2="33.48" width="5.08" layer="1"/>
+<wire x1="43.64" y1="33.48" x2="43.815" y2="33.655" width="5.08" layer="1"/>
 </signal>
 <signal name="RLY-">
