File: PCB Files/Solid-State Sidekick/Solid-State Sidekick v1.brd (EAGLE design)
At the start: 66 x 72.4 mm, 6 parts, among them J1 C14, J2 NEMA, J3 RLY Control, SW1 Rocker

Commit message: Add files via upload
Parts:
- moved J3 1.27 mm to (45.1, 68.6)
Routing:
- net RLY-: track 21.5 -> 20.2 mm
- net RLY+: track 20.9 -> 19.6 mm
Changed lines of the file:
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@@
 </autorouter>
 <elements>
-<element name="J3" library="TimWoo-Connectors" library_urn="urn:adsk.eagle:library:500889" package="SCREWTERMINAL-3.5MM-2" package3d_urn="urn:adsk.eagle:package:501344/1" value="RLY Control" x="45.085" y="69.85" rot="R180">
-<attribute name="PROD_ID" value="CONN-08399" x="45.085" y="69.85" size="1.778" layer="27" rot="R180" display="off"/>
+<element name="J3" library="TimWoo-Connectors" library_urn="urn:adsk.eagle:library:500889" package="SCREWTERMINAL-3.5MM-2" package3d_urn="urn:adsk.eagle:package:501344/1" value="RLY Control" x="45.085" y="68.58" rot="R180">
+<attribute name="PROD_ID" value="CONN-08399" x="45.085" y="68.58" size="1.778" layer="27" rot="R180" display="off"/>
 </element>
 <element name="J1" library="TimWoo-Connectors" library_urn="urn:adsk.eagle:library:500889" package="703W-00/53" value="C14" x="16.51" y="25.4" rot="R90"/>
@@
 <contactref element="RLY1" pad="2"/>
 <contactref element="J3" pad="2"/>
-<wire x1="41.585" y1="69.85" x2="52.07" y2="59.365" width="0.6096" layer="16"/>
-<wire x1="52.07" y1="59.365" x2="52.07" y2="53.34" width="0.6096" layer="16"/>
+<wire x1="41.585" y1="68.58" x2="52.07" y2="58.095" width="0.6096" layer="16"/>
+<wire x1="52.07" y1="58.095" x2="52.07" y2="53.34" width="0.6096" layer="16"/>
 </signal>
 <signal name="L">
@@
 <vertex x="36.83" y="71.12"/>
 <vertex x="38.1" y="71.12"/>
-<vertex x="38.1" y="69.85"/>
-<vertex x="49.53" y="58.42"/>
+<vertex x="38.1" y="68.58"/>
+<vertex x="49.53" y="57.15"/>
 <vertex x="49.53" y="52.07"/>
 <vertex x="50.8" y="50.8"/>
 <vertex x="58.42" y="50.8"/>
 <vertex x="59.69" y="52.07"/>
-<vertex x="59.69" y="58.42"/>
-<vertex x="48.26" y="69.85"/>
+<vertex x="59.69" y="57.15"/>
+<vertex x="48.26" y="68.58"/>
 <vertex x="48.26" y="71.12"/>
 <vertex x="64.77" y="71.12"/>
@@
 <vertex x="36.83" y="71.12"/>
 <vertex x="38.1" y="71.12"/>
-<vertex x="38.1" y="69.85"/>
-<vertex x="49.53" y="58.42"/>
+<vertex x="38.1" y="68.58"/>
+<vertex x="49.53" y="57.15"/>
 <vertex x="49.53" y="52.07"/>
 <vertex x="50.8" y="50.8"/>
 <vertex x="58.42" y="50.8"/>
 <vertex x="59.69" y="52.07"/>
-<vertex x="59.69" y="58.42"/>
-<vertex x="48.26" y="69.85"/>
+<vertex x="59.69" y="57.15"/>
+<vertex x="48.26" y="68.58"/>
 <vertex x="48.26" y="71.12"/>
 <vertex x="64.77" y="71.12"/>
@@
 <contactref element="RLY1" pad="1"/>
 <contactref element="J3" pad="1"/>
-<wire x1="45.085" y1="69.85" x2="57.15" y2="57.785" width="0.6096" layer="16"/>
-<wire x1="57.15" y1="57.785" x2="57.15" y2="53.34" width="0.6096" layer="16"/>
+<wire x1="45.085" y1="68.58" x2="57.15" y2="56.515" width="0.6096" layer="16"/>
+<wire x1="57.15" y1="56.515" x2="57.15" y2="53.34" width="0.6096" layer="16"/>
 </signal>
 </signals>

Commit message: Add files via upload
Parts:
- moved LOGO1 2.54 mm to (52.1, 5.08), flipped to the top
- moved J2 1.27 mm to (43.2, 25.4)
- moved J3 1.27 mm to (43.8, 68.6)
- moved RLY1 1.27 mm to (41.9, 53.3)
Routing:
- net GND: track 31.3 -> 30.1 mm
Other:
- board size 66 x 72.4 mm -> 63.5 x 72.4 mm
- board text added: "Sidekick v2"
- board text removed: "Solid-State Sidekick v1"
