File: PCB Files/Solid-State Sidekick/Solid-State Sidekick v1.sch (EAGLE design)
At the start: 5 parts, among them J1 C14, J2 NEMA, J3 RLY Control, SW1 Rocker

Commit message: Add files via upload
Parts:
- added LOGO1: OSHW-LOGOL, SparkFun-Aesthetics:OSHW-LOGOL
Changed lines of the file:
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@@
 <?xml version="1.0" encoding="utf-8"?>
 <!DOCTYPE eagle SYSTEM "eagle.dtd">
-<eagle version="8.4.0">
+<eagle version="8.4.1">
 <drawing>
 <settings>
@@
 <part name="GND2" library="TimWoo-Aesthetics" library_urn="urn:adsk.eagle:library:502097" deviceset="GND" device=""/>
 <part name="FRAME2" library="TimWoo-Aesthetics" library_urn="urn:adsk.eagle:library:502097" deviceset="SCHEMATIC_FRAME" device=""/>
+<part name="LOGO1" library="SparkFun-Aesthetics" library_urn="urn:adsk.eagle:library:507" deviceset="OSHW-LOGO" device="L" package3d_urn="urn:adsk.eagle:package:37097/1"/>
 </parts>
 <sheets>
@@
 <instance part="GND2" gate="1" x="66.04" y="2.54"/>
 <instance part="FRAME2" gate="G$2" x="99.06" y="0"/>
+<instance part="LOGO1" gate="G$1" x="111.76" y="45.72"/>
 </instances>
 <busses>
